File: hardware/pcb/Calunium_v2/Calunium_v2.brd (EAGLE design)
At the start: 99.1 x 78.7 mm, 48 parts, among them IC1 MCP1702, IC2 ATMEGA1284, IC3 DS1307, Q1 2N7000, U1 CALUNIUM-SHIELD, X1 PWR, X2 JTAG, X3 UART0, X4 USBPTH, Y1 16MHz, Y2 32k768

Commit message: Updating v2.0 PCB design files.
Parts:
- removed BAT2: CR1220, SparkFun:BATTCON_12MM_PTH
- added C10, C11: 22p, SparkFun:CAP-PTH-SMALL
- added C12, C13, C14: 100n, SparkFun:CAP-PTH-SMALL
- added IC4: ATMEGA1284, SteveMarple:DIL40
- added L1: 10uH, SteveMarple:RES-AXIAL-0.4
- added R8: 100k, SteveMarple:RES-AXIAL-0.4
- added RF1: RFM12B, SteveMarple:RFM12B
- added U$1: MICRO-SD-SOCKETHIROSE-DM3D, SteveMarple:MICRO-SD-SOCKET-HIROSE-DM3D
- added X5: UART0, SparkFun:MOLEX-1X6-RA_LOCK
- C4: value 4u7 -> 100p; device SparkFun:CPOL-RADIAL-10UF-25V -> SparkFun:CAP-PTH-SMALL
- C6: value 100n -> 4u7; device SparkFun:CAP-PTH-SMALL -> SparkFun:CPOL-RADIAL-10UF-25V
- C8: value 22p -> 1u; device SparkFun:CAP-PTH-SMALL -> SparkFun:CAP-PTH-5MM
- C9: value 22p -> 100n
- D1: value 1N4001 -> BAT85; device SparkFun:DIODE-1N4001 -> SteveMarple:DIODE-TH-0.4
- D2: value (none) -> BAT85; device SparkFun:DIODE-1N4148 -> SteveMarple:DIODE-TH-0.4
- H1, H2, H3, H4: value MOUNT-PAD-ROUND3.0 -> (none)
- IC1: value MCP1702 -> MCP1702-3.3
- IC2: value ATMEGA1284 -> DS1307; device atmel:DIL40 -> SteveMarple:DIL08-SOIC8
- IC3: value DS1307 -> MCP1702-5.0; device SteveMarple:DIL08-SOIC8 -> SteveMarple:TO-92
- JP2: value A4/SDA -> SDA/A4
- JP3: value A5/SCL -> SCL/A5
- JP4: value 3V3/5V -> D6 SQW/RFM12B
- JP5: value SQW D6 -> 3V3/5V; device SparkFun:1X02 -> SparkFun:1X03
- JP6: value AUTO RST -> VREG PWR
- JP7: value FTDI PWR -> AUTO RST
- JP8: value USB PWR -> FTDI PWR
- R4: value 10k -> 4k7
- R6: value 4k7 -> 10k
- R7: value 22R -> 1k
- U1: device SteveMarple:CALUNIUM-SHIELD-NO-OUTLINE-NO-HOLES-V2 -> SteveMarple:CALUNIUM-SHIELD-NO-OUTLINE-NO-HOLES-NO-TEXT-V2
- X3: value UART0 -> USB; device SparkFun:MOLEX-1X6-RA_LOCK -> SteveMarple:USB-B-PTH
- X4: value USBPTH -> CONN-SMATHD; device SteveMarple:USB-B-PTH -> SteveMarple:SMA-THD
- Y1: value 16MHz -> 32k768; device SteveMarple:HC49U-V-RESONATOR -> SteveMarple:TC38H
- Y2: value 32k768 -> 16MHz; device SparkFun:TC38H -> SteveMarple:HC49U-V-RESONATOR
- moved Y2 85.6 mm to (22.9, 66.7)
- moved Y1 85.2 mm to (88.3, 11.4)
- moved C4 83.9 mm to (94.0, 11.4)
- moved R7 69.8 mm to (92.7, 36.8), turned to 90 degrees
- moved IC3 68.7 mm to (22.9, 34.3), turned to 180 degrees
- moved IC2 68.7 mm to (90.2, 20.3), turned to 0 degrees
- moved R3 54.4 mm to (76.2, 42.5), turned to 0 degrees
- moved C3 53.8 mm to (83.8, 24.1)
- moved C8 44.7 mm to (48.3, 25.1), turned to 180 degrees
- moved D2 30.2 mm to (95.9, 36.8), turned to 270 degrees
- moved C6 29.9 mm to (14.0, 38.1)
- moved R6 28.2 mm to (73.0, 61.0), turned to 270 degrees
- moved JP4 27.9 mm to (71.1, 34.3)
- moved C9 27.3 mm to (27.9, 41.9), turned to 0 degrees
- moved JP7 25.4 mm to (7.62, 12.1), turned to 180 degrees
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Connections:
- new net N$11: C4.1, IC2.3, IC2.3@1, R7.P$2
- new net N$14: IC3.3, JP6.1
- new net N$17: RF1.ANT, X4.SIG
- new net RFM12B_!IRQ: JP4.3, RF1.!IRQ
- net !RESET: now also C12.2, D1.A, IC4.9, R6.P$1; no longer C6.2, D2.A, IC2.9, R3.P$1
- net +3V3: now also JP5.1; no longer JP4.1
- net +5V: now also JP5.3, JP6.2; no longer JP4.3
- net +5V_USB: now also X3.VBUS; no longer JP7.2
- net 0(RX0): now also IC4.14, X5.4; no longer IC2.14, X3.4
- net 1(TX0): now also IC4.15, X5.5; no longer IC2.15, X3.5
- net 10: now also IC4.5; no longer IC2.5
- net 11(MOSI): now also IC4.6, RF1.SDI, U$1.CMD; no longer IC2.6
- net 12(MISO): now also IC4.7, RF1.SDO, U$1.DAT0; no longer IC2.7
- net 13(SCK): now also IC4.8, RF1.SCK, U$1.CLK; no longer IC2.8
- net 14: now also IC4.29, R8.P$1, RF1.!SEL; no longer IC2.29
- net 15: now also IC4.28; no longer IC2.28
- net 16(TDI): now also IC4.27; no longer IC2.27
- net 17(TDO): now also IC4.26; no longer IC2.26
- net 18(TMS): now also IC4.25; no longer IC2.25
- net 19(TCK): now also IC4.24; no longer IC2.24
- net 2(RX1): now also IC4.16; no longer IC2.16
- net 20(SDA): now also IC2.5, IC2.5@1, IC4.23, R5.P$1; no longer IC2.23, IC3.5, IC3.5@1, R6.P$1
- net 21(SCL): now also IC2.6, IC2.6@1, IC4.22, R4.P$1; no longer IC2.22, IC3.6, IC3.6@1, R5.P$1
- net 22: now also IC4.18, U$1.CD/DAT3; no longer IC2.18
- net 23: now also IC4.21; no longer IC2.21
- net 3(TX1): now also IC4.17; no longer IC2.17
- net 4: now also IC4.1; no longer IC2.1
- net 5: now also IC4.2; no longer IC2.2
- net 6: now also IC4.3, JP4.2; no longer IC2.3, JP5.2
- net 7: now also IC4.4; no longer IC2.4
- net 8: now also IC4.20; no longer IC2.20
- net 9: now also IC4.19; no longer IC2.19
- net A0: now also IC4.33; no longer IC2.33
- net A1: now also IC4.34; no longer IC2.34
- net A2: now also IC4.35; no longer IC2.35
- net A3: now also IC4.36; no longer IC2.36
- net A4: now also IC4.37; no longer IC2.37
- net A5: now also IC4.38; no longer IC2.38
- net A6: now also IC4.39; no longer IC2.39
- net A7: now also IC4.40; no longer IC2.40
- net AREF: now also C5.1, IC4.32; no longer C3.1, IC2.32
- net AVCC: now also C9.1, IC4.30, L1.P$1; no longer C7.1, IC2.30, R7.P$1
- net GND: now also C10.2, C11.2, C13.2, C14.2, C6.2, IC2.4, IC2.4@1, IC3.1, IC4.11, IC4.31, RF1.GND@0, RF1.GND@1, U$1.GND, U$1.SHIELD@0, X3.GND, X4.GND@0, X4.GND@1, X4.GND@2, X4.GND@3, X5.1, Y2.GND; no longer BAT2.GND, D1.A, IC2.11, IC2.31, IC3.4, IC3.4@1, X3.1, X4.GND, Y1.GND
- net N$1: now also C11.1, IC4.13, Y2.2; no longer C9.1, IC2.13, Y1.2
- net N$10: now also JP8.1, X5.3; no longer JP7.1, X3.3
- net N$12: now also IC2.2, IC2.2@1, Y1.1; no longer IC3.2, IC3.2@1, Y2.1
- net N$15: now also JP7.1, X5.6; no longer JP6.1, X3.6
- net N$16: now also C12.1, JP7.2; no longer C6.1, JP6.2
- net N$2: now also C10.1, IC4.12, Y2.1; no longer C8.1, IC2.12, Y1.1
- net N$5: now also IC2.1, IC2.1@1, Y1.2; no longer IC3.1, IC3.1@1, Y2.2
- net N$9: now also D2.C, R7.P$1; no longer JP8.1, X4.VBUS
- net SQW: now also IC2.7, IC2.7@1, JP4.1, R3.P$1; no longer IC3.7, IC3.7@1, JP5.1, R4.P$1
- net VBATT: now also D2.A; no longer BAT2.VCC@1, IC3.3, IC3.3@1
- net VCC: now also C13.1, C14.1, C3.1, C6.1, C7.1, IC2.8, IC2.8@1, IC4.10, JP5.2, L1.P$2, R8.P$2, RF1.VDD, U$1.VDD; no longer C4.1, C5.1, D2.C, IC2.10, IC3.8, IC3.8@1, JP4.2, R7.P$2
- net VIN: now also C8.1, IC3.2
Routing:
- net 13(SCK): track 107.9 -> 260.9 mm
- net 12(MISO): track 58.9 -> 164.6 mm, vias 2 -> 3
- net 11(MOSI): track 79.5 -> 176.8 mm, vias 1 -> 0
- net VCC: track 228.5 -> 284.4 mm, vias 0 -> 2
- net GND: track 447.7 -> 502.9 mm, vias 0 -> 4
- net 22: track 73.9 -> 124.1 mm, vias 0 -> 1
- net !RESET: track 153.3 -> 196.1 mm, vias 1 -> 0
- net SQW: track 23.6 -> 60.6 mm
- net N$11: track 0.00 -> 36.1 mm
- net VIN: track 7.62 -> 39.7 mm, vias 0 -> 1
- net VBATT: track 160.9 -> 129.7 mm, vias 1 -> 0
- net 1(TX0): track 144.0 -> 114.8 mm, vias 2 -> 1
- net RFM12B_!IRQ: track 0.00 -> 25.1 mm
- net 6: track 67.6 -> 48.8 mm
- net A5: track 36.5 -> 18.4 mm, vias 0 -> 1
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- added copper zone on layer 1, net GND
- added copper zone on layer 16, net GND
Other:
- board text added: "!RESET"
- board text added: "0"
- board text added: "1"
- board text added: "10"
- board text added: "11"
- board text added: "12"
- board text added: "13"
- board text added: "14"
- board text added: "15"
- board text added: "16"
- board text added: "17"
- board text added: "18"
- board text added: "19"
- board text added: "2"
- board text added: "20"
- board text added: "21"
- board text added: "22"
- board text added: "23"
- board text added: "3"
- board text added: "3V3"
- board text added: "4"
- board text added: "5"
- board text added: "5V"
- board text added: "6"
- board text added: "7"
- board text added: "8"
- board text added: "9"
- board text added: ">PLOT_DATE_TIME"
- board text added: "A0"
- board text added: "A1"
- board text added: "A2"
- board text added: "A3"
- board text added: "A4"
- board text added: "A5"
- board text added: "A6"
- board text added: "A7"
- board text added: "AREF"
- board text added: "IOREF"
- board text added: "MHz"
- board text added: "NC"
- board text added: "RX0"
- board text added: "RX1"
- board text added: "S/N"
- board text added: "SCL"
- board text added: "SDA"
- board text added: "TX0"
- board text added: "TX1"
- board text added: "Vin"
- board text removed: "(A4)"
- board text removed: "(A5)"
- board text removed: ">LAST_DATE_TIME"
- board text removed: "Add S/N, XTAL rectangles to underside"
- board text removed: "PRELIMINARY"
