File: hardware/pcb/Calunium_v2/Calunium_v2.sch (EAGLE design)
At the start: 48 parts, among them IC1 MCP1702, IC2 ATMEGA1284, IC3 DS1307, Q1 2N7000, U1 CALUNIUM-SHIELD, X1 PWR, X2 JTAG, X3 UART0, X4 USBPTH, Y1 16MHz, Y2 32k768

Commit message: Updating v2.0 PCB design files.
Parts:
- removed BAT2: CR1220, SparkFun:BATTERY12PTH
- added C10, C11: 22p, SparkFun:CAPPTH
- added C12, C13, C14: 100n, SparkFun:CAPPTH
- added IC4: ATMEGA1284, SteveMarple:ATMEGA644-20PU
- added L1: 10uH, SteveMarple:INDUCTOR0.4"-AXIAL
- added R8: 100k, SteveMarple:RESISTOR
- added RF1: RFM12B, SteveMarple:RFM12BSMD
- added U$1: MICRO-SD-SOCKETHIROSE-DM3D, SteveMarple:MICRO-SD-SOCKETHIROSE-DM3D
- added X5: UART0, SparkFun:ARDUINO_SERIAL_PROGRAMRA_LOCK
- C4: value 4u7 -> 100p; device SparkFun:CAP_POLPTH2 -> SparkFun:CAPPTH
- C6: value 100n -> 4u7; device SparkFun:CAPPTH -> SparkFun:CAP_POLPTH2
- C8: value 22p -> 1u; device SparkFun:CAPPTH -> SparkFun:CAPPTH1
- C9: value 22p -> 100n
- D1: value 1N4001 -> BAT85; device SparkFun:DIODEPTH -> SteveMarple:DIODE-SCHOTTKY
- D2: value (none) -> BAT85; device SparkFun:DIODE1N4148 -> SteveMarple:DIODE-SCHOTTKY
- IC1: value MCP1702 -> MCP1702-3.3
- IC2: value ATMEGA1284 -> DS1307; device atmel:ATMEGA644-20PU -> SteveMarple:DS1307DIL08/SOIC8
- IC3: value DS1307 -> MCP1702-5.0; device SteveMarple:DS1307DIL08/SOIC8 -> SteveMarple:MCP1702
- JP2: value A4/SDA -> SDA/A4
- JP3: value A5/SCL -> SCL/A5
- JP4: value 3V3/5V -> D6 SQW/RFM12B
- JP5: value SQW D6 -> 3V3/5V; device SparkFun:JUMPER-2PTH -> SparkFun:JUMPER-3PTH
- JP6: value AUTO RST -> VREG PWR
- JP7: value FTDI PWR -> AUTO RST
- JP8: value USB PWR -> FTDI PWR
- R4: value 10k -> 4k7
- R6: value 4k7 -> 10k
- R7: value 22R -> 1k
- U1: device SteveMarple:CALUNIUM-SHIELD-V2 -> SteveMarple:CALUNIUM-SHIELD-V2NO-OUTLINE-NO-HOLES-NO-TEXT
- X3: value UART0 -> USB; device SparkFun:ARDUINO_SERIAL_PROGRAMRA_LOCK -> SteveMarple:USBPTH
- X4: value USBPTH -> CONN-SMATHD; device SteveMarple:USBPTH -> SteveMarple:CONN-SMATHD
- Y1: value 16MHz -> 32k768; device SteveMarple:CRYSTAL-RESONATOR -> SteveMarple:CRYSTALTC38H
- Y2: value 32k768 -> 16MHz; device SparkFun:CRYSTALTC38H -> SteveMarple:CRYSTAL-RESONATOR; OPTION (none) -> Crystal or ceramic resonator. Max 12MHz for 3V3 operation.
Connections:
- new net N$11: C4.1, IC2.VBATT, R7.2
- new net N$14: IC3.VOUT, JP6.1
- new net N$17: RF1.ANT, X4.SIGNAL
- new net RFM12B_!IRQ: JP4.3, RF1.!IRQ
- net !RESET: now also C12.2, D1.A, IC4.!RESET, R6.1; no longer C6.2, D2.A, IC2.!RESET, R3.1
- net +3V3: now also JP5.1; no longer JP4.1
- net +5V: now also JP5.3, JP6.2; no longer JP4.3
- net +5V_USB: now also X3.VBUS; no longer JP7.2
- net 0(RX0): now also IC4.PCINT24/RXD0_PD0, X5.TXO; no longer IC2.PCINT24/RXD0_PD0, X3.TXO
- net 1(TX0): now also IC4.PCINT25/TXD0_PD1, X5.RXI; no longer IC2.PCINT25/TXD0_PD1, X3.RXI
- net 10: now also IC4.PCINT12/OC0B/SS_PB4; no longer IC2.PCINT12/OC0B/SS_PB4
- net 11(MOSI): now also IC4.PCINT13/MOSI_PB5, RF1.SDI, U$1.CMD; no longer IC2.PCINT13/MOSI_PB5
- net 12(MISO): now also IC4.PCINT14/MISO_PB6, RF1.SDO, U$1.DAT0; no longer IC2.PCINT14/MISO_PB6
- net 13(SCK): now also IC4.PCINT15/SCK_PB7, RF1.SCK, U$1.CLK; no longer IC2.PCINT15/SCK_PB7
- net 14: now also IC4.PCINT23/TOSC2_PC7, R8.1, RF1.!SEL; no longer IC2.PCINT23/TOSC2_PC7
- net 15: now also IC4.PCINT22/TOSC1_PC6; no longer IC2.PCINT22/TOSC1_PC6
- net 16(TDI): now also IC4.PCINT21/TDI_PC5; no longer IC2.PCINT21/TDI_PC5
- net 17(TDO): now also IC4.PCINT20/TDO_PC4; no longer IC2.PCINT20/TDO_PC4
- net 18(TMS): now also IC4.PCINT19/TMS_PC3; no longer IC2.PCINT19/TMS_PC3
- net 19(TCK): now also IC4.PCINT18/TCK_PC2; no longer IC2.PCINT18/TCK_PC2
- net 2(RX1): now also IC4.PCINT26/INT0_PD2; no longer IC2.PCINT26/INT0_PD2
- net 20(SDA): now also IC2.SDA, IC4.PCINT17/SDA_PC1, R5.1; no longer IC2.PCINT17/SDA_PC1, IC3.SDA, R6.1
- net 21(SCL): now also IC2.SCL, IC4.PCINT16/SCL_PC0, R4.1; no longer IC2.PCINT16/SCL_PC0, IC3.SCL, R5.1
- net 22: now also IC4.PCINT28/OC1B_PD4, U$1.CD/DAT3; no longer IC2.PCINT28/OC1B_PD4
- net 23: now also IC4.PCINT31/OC2A_PD7; no longer IC2.PCINT31/OC2A_PD7
- net 3(TX1): now also IC4.PCINT27/INT1_PD3; no longer IC2.PCINT27/INT1_PD3
- net 4: now also IC4.PCINT8/XCK0/T0_PB0; no longer IC2.PCINT8/XCK0/T0_PB0
- net 5: now also IC4.PCINT9/CLKO/T1_PB1; no longer IC2.PCINT9/CLKO/T1_PB1
- net 6: now also IC4.PCINT10/INT2/AIN0_PB2, JP4.2; no longer IC2.PCINT10/INT2/AIN0_PB2, JP5.2
- net 7: now also IC4.PCINT11/OC0A/AIN1_PB3; no longer IC2.PCINT11/OC0A/AIN1_PB3
- net 8: now also IC4.PCINT30/OC2B/ICP_PD6; no longer IC2.PCINT30/OC2B/ICP_PD6
- net 9: now also IC4.PCINT29/OC1A_PD5; no longer IC2.PCINT29/OC1A_PD5
- net A0: now also IC4.PCINT7/ADC7_PA7; no longer IC2.PCINT7/ADC7_PA7
- net A1: now also IC4.PCINT6/ADC6_PA6; no longer IC2.PCINT6/ADC6_PA6
- net A2: now also IC4.PCINT5/ADC5_PA5; no longer IC2.PCINT5/ADC5_PA5
- net A3: now also IC4.PCINT4/ADC4_PA4; no longer IC2.PCINT4/ADC4_PA4
- net A4: now also IC4.PCINT3/ADC3_PA3; no longer IC2.PCINT3/ADC3_PA3
- net A5: now also IC4.PCINT2/ADC2_PA2; no longer IC2.PCINT2/ADC2_PA2
- net A6: now also IC4.PCINT1/ADC1_PA1; no longer IC2.PCINT1/ADC1_PA1
- net A7: now also IC4.PCINT0/ADC0_PA0; no longer IC2.PCINT0/ADC0_PA0
- net AREF: now also C5.1, IC4.AREF; no longer C3.1, IC2.AREF
- net AVCC: now also C9.1, IC4.AVCC, L1.1; no longer C7.1, IC2.AVCC, R7.1
- net GND: now also C10.2, C11.2, C13.2, C14.2, C4.2, C6.-, IC4.GND, IC4.GND@1, RF1.GND, U$1.SHIELD, U$1.VSS, X5.GND, Y2.2; no longer BAT2.-, C4.-, D1.A, IC2.GND@1, Y1.2
- net N$1: now also C11.1, IC4.XTAL1, Y2.3; no longer C9.1, IC2.XTAL1, Y1.3
- net N$10: now also JP8.1, X5.VCC; no longer JP7.1, X3.VCC
- net N$12: now also IC2.X2, Y1.1; no longer IC3.X2, Y2.1
- net N$15: now also JP7.1, X5.DTR; no longer JP6.1, X3.DTR
- net N$16: now also C12.1, JP7.2; no longer C6.1, JP6.2
- net N$2: now also C10.1, IC4.XTAL2, Y2.1; no longer C8.1, IC2.XTAL2, Y1.1
- net N$5: now also IC2.X1, Y1.2; no longer IC3.X1, Y2.2
- net N$9: now also D2.C, R7.1; no longer JP8.1, X4.VBUS
- net SQW: now also IC2.SQW, JP4.1, R3.1; no longer IC3.SQW, JP5.1, R4.1
- net VBATT: now also D2.A; no longer BAT2.+, IC3.VBATT
- net VCC: now also C13.1, C14.1, C3.1, C6.+, C7.1, IC4.VCC, JP5.2, L1.2, R8.2, RF1.VDD, U$1.VDD; no longer C4.+, C5.1, D2.C, IC3.VCC, JP4.2, R7.2
- net VIN: now also C8.1, IC3.VIN
Other:
- note added: "5V regulator"
- note added: "Omit load capacitors if resonator"
- note added: "Power LED"
- note added: "Pull-up disables RFM12B"
- note added: "RFM12B radio module"
- note added: "USB power"
- note added: "fitted instead of crystal"
- note added: "when ICSP in use"
- note removed: "Alternative"
- note removed: "Check battery footprint"
- note removed: "POWER LED"
- note removed: "TODO: IOREF"
- note removed: "V-USB"
- note removed: "battery holders"
- moved on the sheet: BAT1, C3, C5, C7, C8, C9, F1, H1, H2, H3, H4, JP4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
